Commit message: testing without stearing controller

File: mobile_manipulator_description/urdf/joints.xacro (robot description, xacro)
@@ -61,6 +61,6 @@
   <!-- ============================================ -->
   <!-- Front Right Steering -->
-  <joint name="${frame_prefix}fr_steer_joint" type="revolute">
-  <!-- <joint name="${frame_prefix}fr_steer_joint" type="fixed"> -->
+  <!-- <joint name="${frame_prefix}fr_steer_joint" type="revolute"> -->
+  <joint name="${frame_prefix}fr_steer_joint" type="fixed">
     <origin xyz="${steer_x_offset} ${-steer_y_offset} ${steer_z_offset}" rpy="-1.5708 0 -1.5708"/>
     <parent link="${frame_prefix}base_link"/>
@@ -70,23 +70,29 @@
   </joint>
   <!-- Front Left Steering -->
-  <joint name="${frame_prefix}fl_steer_joint" type="revolute">
-  <!-- <joint name="${frame_prefix}fl_steer_joint" type="fixed"> -->
+  <!-- <joint name="${frame_prefix}fl_steer_joint" type="revolute"> -->
+  <joint name="${frame_prefix}fl_steer_joint" type="fixed">
     <origin xyz="${steer_x_offset} ${steer_y_offset} ${steer_z_offset}" rpy="-1.5708 0 -1.5708"/>
     <parent link="${frame_prefix}base_link"/>
     <child link="${frame_prefix}fl_steer_link"/>
-    <axis xyz="0 1 0"/>
-    <limit lower="-1.571" upper="1.571" effort="100" velocity="10"/>
+    <!-- <axis xyz="0 1 0"/> -->
+    <!-- <limit lower="-1.571" upper="1.571" effort="100" velocity="10"/> -->
   </joint>
   <!-- Back Right Steering (Fixed) -->
+  <!-- <joint name="${frame_prefix}br_steer_joint" type="revolute"> -->
   <joint name="${frame_prefix}br_steer_joint" type="fixed">
     <origin xyz="${-steer_x_offset} ${-steer_y_offset} ${steer_z_offset}" rpy="-1.5708 0 -1.5708"/>
     <parent link="${frame_prefix}base_link"/>
     <child link="${frame_prefix}br_steer_link"/>
+    <!-- <axis xyz="0 1 0"/> -->
+    <!-- <limit lower="-1.571" upper="1.571" effort="100" velocity="10"/> -->
   </joint>
   <!-- Back Left Steering (Fixed) -->
+  <!-- <joint name="${frame_prefix}bl_steer_joint" type="revolute"> -->
   <joint name="${frame_prefix}bl_steer_joint" type="fixed">
     <origin xyz="${-steer_x_offset} ${steer_y_offset} ${steer_z_offset}" rpy="-1.5708 0 -1.5708"/>
     <parent link="${frame_prefix}base_link"/>
     <child link="${frame_prefix}bl_steer_link"/>
+    <!-- <axis xyz="0 1 0"/> -->
+    <!-- <limit lower="-1.571" upper="1.571" effort="100" velocity="10"/> -->
   </joint>
   <!-- ============================================ -->

File: mobile_manipulator_description/urdf/mobile_manipulator.urdf.xacro (robot description, xacro)
@@ -10,5 +10,5 @@
   <xacro:include filename="$(find mobile_manipulator_description)/urdf/joints.xacro"/>
   <xacro:include filename="$(find mobile_manipulator_description)/urdf/mobile_manipulator_ros2_control.xacro"/>
-  <xacro:include filename="$(find mobile_manipulator_description)/urdf/sensors.xacro"/>
   <xacro:include filename="$(find mobile_manipulator_description)/urdf/mobile_manipulator_gazebo.xacro"/>
+  <!-- <xacro:include filename="$(find mobile_manipulator_description)/urdf/sensors.xacro"/> -->
 </robot>

File: mobile_manipulator_description/urdf/mobile_manipulator_ros2_control.xacro (robot description, xacro)
@@ -22,6 +22,6 @@
       <joint name="${frame_prefix}bl_wheel_joint">
         <command_interface name="velocity">
-          <param name="min">-200.0</param>  <!-- Increased -->
-          <param name="max">200.0</param>   <!-- Increased -->
+          <param name="min">-200.0</param>
+          <param name="max">200.0</param>
         </command_interface>
         <state_interface name="position"/>
@@ -53,5 +53,5 @@
       </joint>
       <!-- STEERING POSITION CONTROLLERS -->
-      <joint name="${frame_prefix}fl_steer_joint">
+      <!-- <joint name="${frame_prefix}fl_steer_joint">
         <command_interface name="position">
           <param name="min">-1.571</param>
@@ -60,6 +60,6 @@
         <state_interface name="position"/>
         <state_interface name="velocity"/>
-      </joint>
-      <joint name="${frame_prefix}fr_steer_joint">
+      </joint> -->
+      <!-- <joint name="${frame_prefix}fr_steer_joint">
         <command_interface name="position">
           <param name="min">-1.571</param>
@@ -68,5 +68,5 @@
         <state_interface name="position"/>
         <state_interface name="velocity"/>
-      </joint>
+      </joint> -->
       <!-- UR ARM JOINTS remain unchanged -->
       <joint name="${frame_prefix}ur_joint1">
